File: balancer.kicad_pcb (KiCad board)
At the start: 2 copper layers, 50 x 50 mm, 54 parts, among them IC1 TLV3404, IC2 MAX923, IC3 MAX923, IC4 MAX923, J1 S4B-XH-SM4-TB, J2 Output (+), J3 Output (-), J4 Input (+), J5 Input (-), Q1 IRF7455PBF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

Commit message: updated pull ups on quad comparator to 1M, update center divider resistor to 340K to be closer to 4.2V charge cutoff
Parts:
- R1, R2: value 10M -> 1M
- R14, R21, R7: value 332K -> 340K
Changed lines of the file:
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@@
       (effects (font (size 1 1) (thickness 0.15)) (justify mirror))
     )
-    (fp_text value 10M (at 0 -1.75 270) (layer B.Fab)
+    (fp_text value 1M (at 0 -1.75 270) (layer B.Fab)
       (effects (font (size 1 1) (thickness 0.15)) (justify mirror))
     )
@@
       (effects (font (size 1 1) (thickness 0.15)) (justify mirror))
     )
-    (fp_text value 10M (at 0 -1.75 180) (layer B.Fab)
+    (fp_text value 1M (at 0 -1.75 180) (layer B.Fab)
       (effects (font (size 1 1) (thickness 0.15)) (justify mirror))
     )
@@
       (effects (font (size 1 1) (thickness 0.15)))
     )
-    (fp_text value 332K (at 0 1.75 300) (layer F.Fab)
+    (fp_text value 340K (at 0 1.75 300) (layer F.Fab)
       (effects (font (size 1 1) (thickness 0.15)))
     )
@@
       (effects (font (size 1 1) (thickness 0.15)))
     )
-    (fp_text value 332K (at 0 1.75 180) (layer F.Fab)
+    (fp_text value 340K (at 0 1.75 180) (layer F.Fab)
       (effects (font (size 1 1) (thickness 0.15)))
     )
@@
       (effects (font (size 1 1) (thickness 0.15)))
     )
-    (fp_text value 332K (at 0 1.75 60) (layer F.Fab)
-      (effects (font (size 1 1) (thickness 0.15)))
-    )
+    (fp_text value 340K (at 0 1.75 60) (layer F.Fab)
+      (effects (font (size 1 1) (thickness 0.15)))
+    )
